Commit message: Add Gazebo simulation support for SO-ARM100
Spawn the SO-ARM100 in Gazebo Harmonic with ros2_control:

- Add gz_ros2_control plugin and ros2_control joint definitions to URDF
- Add gazebo.launch.py to spawn robot, bridge clock, and load controllers
- Add controllers.yaml with joint_state_broadcaster and arm_controller
- Add gazebo.xacro with link friction coefficients
- Add empty.world with ground plane and sun
- Install worlds directory in CMakeLists

File: urdf/so100.urdf.xacro (robot description, xacro)
@@ -3,11 +3,11 @@
        name="so100">
   <!-- ========================================================= -->
-  <!-- Materials                                                  -->
-  <!-- ========================================================= -->
-  <material name="so100_gray">
-    <color rgba="0.65 0.65 0.65 1.0"/>
+  <!-- MATERIALS                                                  -->
+  <!-- ========================================================= -->
+  <material name="so100_white">
+    <color rgba="0.92 0.92 0.92 1.0"/>
   </material>
-  <material name="so100_dark">
-    <color rgba="0.15 0.15 0.15 1.0"/>
+  <material name="so100_black">
+    <color rgba="0.03 0.03 0.03 1.0"/>
   </material>
   <!-- ========================================================= -->
@@ -15,29 +15,4 @@
   <!-- ========================================================= -->
   <link name="base">
-    <!-- Main base -->
-    <visual>
-      <geometry>
-        <mesh filename="package://so100_description/meshes/so100/Base.stl"/>
-      </geometry>
-      <material name="so100_gray"/>
-    </visual>
-    <!-- Base motor -->
-    <visual>
-      <geometry>
-        <mesh filename="package://so100_description/meshes/so100/Base_Motor.stl"/>
-      </geometry>
-      <material name="so100_dark"/>
-    </visual>
-    <!-- Collision -->
-    <collision>
-      <geometry>
-        <mesh filename="package://so100_description/meshes/so100/Base.stl"/>
-      </geometry>
-    </collision>
-    <collision>
-      <geometry>
-        <mesh filename="package://so100_description/meshes/so100/Base_Motor.stl"/>
-      </geometry>
-    </collision>
     <inertial>
       <mass value="1.0"/>
@@ -51,4 +26,21 @@
         izz="0.01"/>
     </inertial>
+    <visual>
+      <geometry>
+        <mesh filename="package://so100_description/meshes/so100/Base.stl"/>
+      </geometry>
+      <material name="so100_white"/>
+    </visual>
+    <visual>
+      <geometry>
+        <mesh filename="package://so100_description/meshes/so100/Base_Motor.stl"/>
+      </geometry>
+      <material name="so100_black"/>
+    </visual>
+    <collision>
+      <geometry>
+        <mesh filename="package://so100_description/meshes/so100/Base.stl"/>
+      </geometry>
+    </collision>
   </link>
   <!-- ========================================================= -->
@@ -56,19 +48,29 @@
   <!-- ========================================================= -->
   <link name="shoulder">
-    <!-- Shoulder body -->
+    <inertial>
+      <mass value="0.119226"/>
+      <origin
+        xyz="-9.07886e-05 0.0590972 0.031089"
+        rpy="0 0 0"/>
+      <inertia
+        ixx="5.94278e-05"
+        ixy="0"
+        ixz="0"
+        iyy="5.89975e-05"
+        iyz="0"
+        izz="3.13712e-05"/>
+    </inertial>
     <visual>
       <geometry>
         <mesh filename="package://so100_description/meshes/so100/Rotation_Pitch.stl"/>
       </geometry>
-      <material name="so100_gray"/>
-    </visual>
-    <!-- Shoulder motor -->
+      <material name="so100_white"/>
+    </visual>
     <visual>
       <geometry>
         <mesh filename="package://so100_description/meshes/so100/Rotation_Pitch_Motor.stl"/>
       </geometry>
-      <material name="so100_dark"/>
-    </visual>
-    <!-- Collision -->
+      <material name="so100_black"/>
+    </visual>
     <collision>
       <geometry>
@@ -76,22 +78,4 @@
       </geometry>
     </collision>
-    <collision>
-      <geometry>
-        <mesh filename="package://so100_description/meshes/so100/Rotation_Pitch_Motor.stl"/>
-      </geometry>
-    </collision>
-    <inertial>
-      <mass value="0.119226"/>
-      <origin
-        xyz="-9.07886e-05 0.0590972 0.031089"
-        rpy="0 0 0"/>
-      <inertia
-        ixx="5.94278e-05"
-        ixy="0"
-        ixz="0"
-        iyy="5.89975e-05"
-        iyz="0"
-        izz="3.13712e-05"/>
-    </inertial>
   </link>
   <!-- ========================================================= -->
@@ -115,19 +99,29 @@
   <!-- ========================================================= -->
   <link name="upper_arm">
-    <!-- Upper arm body -->
+    <inertial>
+      <mass value="0.162409"/>
+      <origin
+        xyz="-1.72052e-05 0.0701802 0.00310545"
+        rpy="0 0 0"/>
+      <inertia
+        ixx="0.000213312"
+        ixy="0"
+        ixz="0"
+        iyy="0.000167164"
+        iyz="0"
+        izz="7.01522e-05"/>
+    </inertial>
     <visual>
       <geometry>
         <mesh filename="package://so100_description/meshes/so100/Upper_Arm.stl"/>
       </geometry>
-      <material name="so100_gray"/>
-    </visual>
-    <!-- Upper arm motor -->
+      <material name="so100_white"/>
+    </visual>
     <visual>
       <geometry>
         <mesh filename="package://so100_description/meshes/so100/Upper_Arm_Motor.stl"/>
       </geometry>
-      <material name="so100_dark"/>
-    </visual>
-    <!-- Collision -->
+      <material name="so100_black"/>
+    </visual>
     <collision>
       <geometry>
@@ -135,22 +129,4 @@
       </geometry>
     </collision>
-    <collision>
-      <geometry>
-        <mesh filename="package://so100_description/meshes/so100/Upper_Arm_Motor.stl"/>
-      </geometry>
-    </collision>
-    <inertial>
-      <mass value="0.162409"/>
-      <origin
-        xyz="-1.72052e-05 0.0701802 0.00310545"
-        rpy="0 0 0"/>
-      <inertia
-        ixx="0.000213312"
-        ixy="0"
-        ixz="0"
-        iyy="0.000167164"
-        iyz="0"
-        izz="7.01522e-05"/>
-    </inertial>
   </link>
   <!-- ========================================================= -->
@@ -164,6 +140,7 @@
       rpy="-1.8 0 0"/>
     <axis xyz="1 0 0"/>
-    <limit
-      lower="0"
+    <!-- Small tolerance for floating point zero -->
+    <limit
+      lower="-0.001"
       upper="3.5"
       effort="35"
@@ -174,19 +151,29 @@
   <!-- ========================================================= -->
   <link name="lower_arm">
-    <!-- Lower arm body -->
+    <inertial>
+      <mass value="0.147968"/>
+      <origin
+        xyz="-0.00339604 0.00137796 0.0768007"
+        rpy="0 0 0"/>
+      <inertia
+        ixx="0.000138803"
+        ixy="0"
+        ixz="0"
+        iyy="0.000107748"
+        iyz="0"
+        izz="4.84242e-05"/>
+    </inertial>
     <visual>
       <geometry>
         <mesh filename="package://so100_description/meshes/so100/Lower_Arm.stl"/>
       </geometry>
-      <material name="so100_gray"/>
-    </visual>
-    <!-- Lower arm motor -->
+      <material name="so100_white"/>
+    </visual>
     <visual>
       <geometry>
         <mesh filename="package://so100_description/meshes/so100/Lower_Arm_Motor.stl"/>
       </geometry>
-      <material name="so100_dark"/>
-    </visual>
-    <!-- Collision -->
+      <material name="so100_black"/>
+    </visual>
     <collision>
       <geometry>
@@ -194,25 +181,7 @@
       </geometry>
     </collision>
-    <collision>
-      <geometry>
-        <mesh filename="package://so100_description/meshes/so100/Lower_Arm_Motor.stl"/>
-      </geometry>
-    </collision>
-    <inertial>
-      <mass value="0.147968"/>
-      <origin
-        xyz="-0.00339604 0.00137796 0.0768007"
-        rpy="0 0 0"/>
-      <inertia
-        ixx="0.000138803"
-        ixy="0"
-        ixz="0"
-        iyy="0.000107748"
-        iyz="0"
-        izz="4.84242e-05"/>
-    </inertial>
-  </link>
-  <!-- ========================================================= -->
-  <!-- ELBOW FLEX                                                -->
+  </link>
+  <!-- ========================================================= -->
+  <!-- ELBOW FLEX                                                 -->
   <!-- ========================================================= -->
   <joint name="elbow_flex" type="revolute">
@@ -223,7 +192,8 @@
       rpy="1.57079 0 0"/>
     <axis xyz="1 0 0"/>
+    <!-- Small tolerance for floating point zero -->
     <limit
       lower="-3.14158"
-      upper="0"
+      upper="0.001"
       effort="35"
       velocity="1"/>
@@ -233,19 +203,29 @@
   <!-- ========================================================= -->
   <link name="wrist">
-    <!-- Wrist body -->
+    <inertial>
+      <mass value="0.0661321"/>
+      <origin
+        xyz="-0.00852653 -0.0352279 -2.34622e-05"
+        rpy="0 0 0"/>
+      <inertia
+        ixx="3.45403e-05"
+        ixy="0"
+        ixz="0"
+        iyy="2.39041e-05"
+        iyz="0"
+        izz="1.94704e-05"/>
+    </inertial>
     <visual>
       <geometry>
         <mesh filename="package://so100_description/meshes/so100/Wrist_Pitch_Roll.stl"/>
       </geometry>
-      <material name="so100_gray"/>
-    </visual>
-    <!-- Wrist motor -->
+      <material name="so100_white"/>
+    </visual>
     <visual>
       <geometry>
         <mesh filename="package://so100_description/meshes/so100/Wrist_Pitch_Roll_Motor.stl"/>
       </geometry>
-      <material name="so100_dark"/>
-    </visual>
-    <!-- Collision -->
+      <material name="so100_black"/>
+    </visual>
     <collision>
       <geometry>
@@ -253,22 +233,4 @@
       </geometry>
     </collision>
-    <collision>
-      <geometry>
-        <mesh filename="package://so100_description/meshes/so100/Wrist_Pitch_Roll_Motor.stl"/>
-      </geometry>
-    </collision>
-    <inertial>
-      <mass value="0.0661321"/>
-      <origin
-        xyz="-0.00852653 -0.0352279 -2.34622e-05"
-        rpy="0 0 0"/>
-      <inertia
-        ixx="3.45403e-05"
-        ixy="0"
-        ixz="0"
-        iyy="2.39041e-05"
-        iyz="0"
-        izz="1.94704e-05"/>
-    </inertial>
   </link>
   <!-- ========================================================= -->
@@ -289,45 +251,32 @@
   </joint>
   <!-- ========================================================= -->
-  <!-- GRIPPER HOUSING                                            -->
+  <!-- GRIPPER                                                    -->
   <!-- ========================================================= -->
   <link name="gripper">
-    <!-- Fixed jaw body -->
+    <inertial>
+      <mass value="0.0929859"/>
+      <origin
+        xyz="0.00552377 -0.0280167 0.000483583"
+        rpy="0 0 0"/>
+      <inertia
+        ixx="5.03136e-05"
+        ixy="0"
+        ixz="0"
+        iyy="4.64098e-05"
+        iyz="0"
+        izz="2.72961e-05"/>
+    </inertial>
     <visual>
       <geometry>
         <mesh filename="package://so100_description/meshes/so100/Fixed_Jaw.stl"/>
       </geometry>
-      <material name="so100_gray"/>
-    </visual>
-    <!-- Fixed jaw motor -->
+      <material name="so100_white"/>
+    </visual>
     <visual>
       <geometry>
         <mesh filename="package://so100_description/meshes/so100/Fixed_Jaw_Motor.stl"/>
       </geometry>
-      <material name="so100_dark"/>
-    </visual>
-    <!-- Collision -->
-    <collision>
-      <geometry>
-        <mesh filename="package://so100_description/meshes/so100/Fixed_Jaw.stl"/>
-      </geometry>
-    </collision>
-    <collision>
-      <geometry>
-        <mesh filename="package://so100_description/meshes/so100/Fixed_Jaw_Motor.stl"/>
-      </geometry>
-    </collision>
-    <inertial>
-      <mass value="0.0929859"/>
-      <origin
-        xyz="0.00552377 -0.0280167 0.000483583"
-        rpy="0 0 0"/>
-      <inertia
-        ixx="5.03136e-05"
-        ixy="0"
-        ixz="0"
-        iyy="4.64098e-05"
-        iyz="0"
-        izz="2.72961e-05"/>
-    </inertial>
+      <material name="so100_black"/>
+    </visual>
   </link>
   <!-- ========================================================= -->
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